File: Nixie-ProtoBoard.kicad_pcb (KiCad board)
At the start: 4 copper layers, 238.8 x 76.2 mm, 90 parts, among them IC1 ATmega328, J1 Conn_LED, J2 Conn_FTDI, J3 CE_Header_Narrow, J4 Conn_PWR_Ext, Q1 MJE18008-D, SW1 SW_DIP_x01, U1 MCP23017-E_SP, U2 MCP23017-E_SP, U3 MCP23017-E_SP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

Commit message: Minor updates
Parts:
- moved C5 46.7 mm to (246.6, 106.2)
- moved H2 46.7 mm to (254.3, 66.5)
- moved H4 46.7 mm to (254.3, 132.6)
- moved NT11 46.7 mm to (218.7, 104.2)
- moved R20 46.7 mm to (215.1, 71.0)
- moved VTR1 46.7 mm to (254.3, 102.1)
- moved C1 46.7 mm to (206.6, 71.5)
- moved C2 46.7 mm to (125.0, 67.8)
- moved C3 46.7 mm to (125.0, 72.9)
- moved C6 46.7 mm to (256.8, 75.2)
- moved C7 46.7 mm to (242.6, 135.4)
- moved C8 46.7 mm to (251.7, 123.7)
- moved D1 46.7 mm to (194.6, 71.6)
- moved H1 46.7 mm to (25.7, 66.5)
- moved H3 46.7 mm to (25.7, 132.6)
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